File: Mosfetboard.brd (EAGLE design)
At the start: 38.1 x 44.5 mm, 26 parts, among them U1 3.3v

Commit message: add values to resistors
Parts:
- C1: value (none) -> 100n
- R1, R6, R7, R8, R9: value (none) -> 1k
- R2, R3, R4, R5: value (none) -> 10k
Changed lines of the file:
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@@
 <layer number="26" name="bNames" color="7" fill="1" visible="yes" active="yes"/>
 <layer number="27" name="tValues" color="7" fill="1" visible="yes" active="yes"/>
-<layer number="28" name="bValues" color="7" fill="1" visible="no" active="yes"/>
+<layer number="28" name="bValues" color="7" fill="1" visible="yes" active="yes"/>
 <layer number="29" name="tStop" color="7" fill="3" visible="no" active="yes"/>
 <layer number="30" name="bStop" color="7" fill="6" visible="no" active="yes"/>
@@
 <attribute name="VALUE" x="31.323" y="33.4375" size="0.635" layer="28" ratio="10" rot="MR180"/>
 </element>
-<element name="R1" library="simple-shiled" library_urn="urn:adsk.eagle:library:80055" package="0805" package3d_urn="urn:adsk.eagle:package:103226/5" value=" " x="33.02" y="36.83" smashed="yes" rot="MR180">
+<element name="R1" library="simple-shiled" library_urn="urn:adsk.eagle:library:80055" package="0805" package3d_urn="urn:adsk.eagle:package:103226/5" value="1k" x="33.02" y="36.83" smashed="yes" rot="MR180">
 <attribute name="NAME" x="33.02" y="35.941" size="0.6096" layer="26" font="vector" ratio="20" rot="MR180" align="bottom-center"/>
 <attribute name="PROD_ID" value=" " x="33.02" y="36.83" size="1.778" layer="28" rot="MR180" display="off"/>
 <attribute name="VALUE" x="33.02" y="37.719" size="0.6096" layer="28" font="vector" ratio="20" rot="MR180" align="top-center"/>
 </element>
-<element name="R2" library="simple-shiled" library_urn="urn:adsk.eagle:library:80055" package="0805" package3d_urn="urn:adsk.eagle:package:103226/5" value=" " x="25.4" y="16.51" smashed="yes" rot="MR270">
+<element name="R2" library="simple-shiled" library_urn="urn:adsk.eagle:library:80055" package="0805" package3d_urn="urn:adsk.eagle:package:103226/5" value="10k" x="25.4" y="16.51" smashed="yes" rot="MR270">
 <attribute name="NAME" x="24.511" y="16.51" size="0.6096" layer="26" font="vector" ratio="20" rot="MR270" align="bottom-center"/>
 <attribute name="PROD_ID" value=" " x="25.4" y="16.51" size="1.778" layer="28" rot="MR270" display="off"/>
 <attribute name="VALUE" x="26.289" y="16.51" size="0.6096" layer="28" font="vector" ratio="20" rot="MR270" align="top-center"/>
 </element>
-<element name="R3" library="simple-shiled" library_urn="urn:adsk.eagle:library:80055" package="0805" package3d_urn="urn:adsk.eagle:package:103226/5" value=" " x="16.51" y="5.08" smashed="yes" rot="MR180">
+<element name="R3" library="simple-shiled" library_urn="urn:adsk.eagle:library:80055" package="0805" package3d_urn="urn:adsk.eagle:package:103226/5" value="10k" x="16.51" y="5.08" smashed="yes" rot="MR180">
 <attribute name="NAME" x="15.24" y="5.461" size="0.6096" layer="26" font="vector" ratio="20" rot="MR180" align="bottom-center"/>
 <attribute name="PROD_ID" value=" " x="16.51" y="5.08" size="1.778" layer="28" rot="MR180" display="off"/>
 <attribute name="VALUE" x="16.51" y="5.969" size="0.6096" layer="28" font="vector" ratio="20" rot="MR180" align="top-center"/>
 </element>
-<element name="R4" library="simple-shiled" library_urn="urn:adsk.eagle:library:80055" package="0805" package3d_urn="urn:adsk.eagle:package:103226/5" value=" " x="17.78" y="16.51" smashed="yes" rot="MR270">
+<element name="R4" library="simple-shiled" library_urn="urn:adsk.eagle:library:80055" package="0805" package3d_urn="urn:adsk.eagle:package:103226/5" value="10k" x="17.78" y="16.51" smashed="yes" rot="MR270">
 <attribute name="NAME" x="16.891" y="16.51" size="0.6096" layer="26" font="vector" ratio="20" rot="MR270" align="bottom-center"/>
 <attribute name="PROD_ID" value=" " x="17.78" y="16.51" size="1.778" layer="28" rot="MR270" display="off"/>
 <attribute name="VALUE" x="18.669" y="16.51" size="0.6096" layer="28" font="vector" ratio="20" rot="MR270" align="top-center"/>
 </element>
-<element name="R5" library="simple-shiled" library_urn="urn:adsk.eagle:library:80055" package="0805" package3d_urn="urn:adsk.eagle:package:103226/5" value=" " x="21.59" y="16.51" smashed="yes" rot="MR270">
+<element name="R5" library="simple-shiled" library_urn="urn:adsk.eagle:library:80055" package="0805" package3d_urn="urn:adsk.eagle:package:103226/5" value="10k" x="21.59" y="16.51" smashed="yes" rot="MR270">
 <attribute name="NAME" x="20.701" y="16.51" size="0.6096" layer="26" font="vector" ratio="20" rot="MR270" align="bottom-center"/>
 <attribute name="PROD_ID" value=" " x="21.59" y="16.51" size="1.778" layer="28" rot="MR270" display="off"/>
 <attribute name="VALUE" x="22.479" y="16.51" size="0.6096" layer="28" font="vector" ratio="20" rot="MR270" align="top-center"/>
 </element>
-<element name="C1" library="simple-shiled" library_urn="urn:adsk.eagle:library:80055" package="C1206K" package3d_urn="urn:adsk.eagle:package:878060/2" value="" x="22.86" y="3.81" smashed="yes" rot="R180">
+<element name="C1" library="simple-shiled" library_urn="urn:adsk.eagle:library:80055" package="C1206K" package3d_urn="urn:adsk.eagle:package:878060/2" value="100n" x="22.86" y="3.81" smashed="yes" rot="R180">
 <attribute name="NAME" x="24.46" y="2.71" size="1.016" layer="25" rot="R180"/>
 <attribute name="VALUE" x="24.46" y="5.91" size="1.016" layer="27" rot="R180"/>
@@
 <attribute name="VALUE" x="34.717" y="14.8225" size="0.635" layer="28" ratio="10" rot="MR0"/>
 </element>
-<element name="R6" library="simple-shiled" library_urn="urn:adsk.eagle:library:80055" package="0805" package3d_urn="urn:adsk.eagle:package:103226/5" value=" " x="25.4" y="31.75" smashed="yes" rot="MR180">
+<element name="R6" library="simple-shiled" library_urn="urn:adsk.eagle:library:80055" package="0805" package3d_urn="urn:adsk.eagle:package:103226/5" value="1k" x="25.4" y="31.75" smashed="yes" rot="MR180">
 <attribute name="NAME" x="25.4" y="30.861" size="0.6096" layer="26" font="vector" ratio="20" rot="MR180" align="bottom-center"/>
 <attribute name="PROD_ID" value=" " x="25.4" y="31.75" size="1.778" layer="28" rot="MR180" display="off"/>
 <attribute name="VALUE" x="25.4" y="32.639" size="0.6096" layer="28" font="vector" ratio="20" rot="MR180" align="top-center"/>
 </element>
-<element name="R7" library="simple-shiled" library_urn="urn:adsk.eagle:library:80055" package="0805" package3d_urn="urn:adsk.eagle:package:103226/5" value=" " x="25.4" y="27.94" smashed="yes" rot="MR180">
+<element name="R7" library="simple-shiled" library_urn="urn:adsk.eagle:library:80055" package="0805" package3d_urn="urn:adsk.eagle:package:103226/5" value="1k" x="25.4" y="27.94" smashed="yes" rot="MR180">
 <attribute name="NAME" x="25.4" y="27.051" size="0.6096" layer="26" font="vector" ratio="20" rot="MR180" align="bottom-center"/>
 <attribute name="PROD_ID" value=" " x="25.4" y="27.94" size="1.778" layer="28" rot="MR180" display="off"/>
 <attribute name="VALUE" x="25.4" y="28.829" size="0.6096" layer="28" font="vector" ratio="20" rot="MR180" align="top-center"/>
 </element>
-<element name="R8" library="simple-shiled" library_urn="urn:adsk.eagle:library:80055" package="0805" package3d_urn="urn:adsk.eagle:package:103226/5" value=" " x="25.4" y="24.13" smashed="yes" rot="MR180">
+<element name="R8" library="simple-shiled" library_urn="urn:adsk.eagle:library:80055" package="0805" package3d_urn="urn:adsk.eagle:package:103226/5" value="1k" x="25.4" y="24.13" smashed="yes" rot="MR180">
 <attribute name="NAME" x="25.4" y="23.241" size="0.6096" layer="26" font="vector" ratio="20" rot="MR180" align="bottom-center"/>
 <attribute name="PROD_ID" value=" " x="25.4" y="24.13" size="1.778" layer="28" rot="MR180" display="off"/>
 <attribute name="VALUE" x="25.4" y="25.019" size="0.6096" layer="28" font="vector" ratio="20" rot="MR180" align="top-center"/>
 </element>
-<element name="R9" library="simple-shiled" library_urn="urn:adsk.eagle:library:80055" package="0805" package3d_urn="urn:adsk.eagle:package:103226/5" value=" " x="25.4" y="20.32" smashed="yes" rot="MR180">
+<element name="R9" library="simple-shiled" library_urn="urn:adsk.eagle:library:80055" package="0805" package3d_urn="urn:adsk.eagle:package:103226/5" value="1k" x="25.4" y="20.32" smashed="yes" rot="MR180">
 <attribute name="NAME" x="25.4" y="19.431" size="0.6096" layer="26" font="vector" ratio="20" rot="MR180" align="bottom-center"/>
 <attribute name="PROD_ID" value=" " x="25.4" y="20.32" size="1.778" layer="28" rot="MR180" display="off"/>
